Commit message: update urdf model

File: mycobot_description/urdf/mycobot.xacro (robot description, xacro)
@@ -26,13 +26,12 @@
       <visual>
         <geometry>
-          <mesh filename="package://mycobot_description/meshes/visual/joint1.dae" />
-        </geometry>
-        <origin xyz="0 0 0" rpy="0 0 0" />
-        <material name="white" />
-      </visual>
-      <collision>
-        <geometry>
-          <mesh filename="package://mycobot_description/meshes/visual/joint1.dae" />
-          <!-- <mesh filename="package://mycobot_description/meshes/collision/link1.stl" /> -->
+          <mesh filename="package://mycobot_description/meshes/visual/link1.dae" />
+        </geometry>
+        <origin xyz="0 0 0" rpy="0 0 0" />
+        <material name="white" />
+      </visual>
+      <collision>
+        <geometry>
+          <mesh filename="package://mycobot_description/meshes/collision/link1.stl" />
         </geometry>
         <origin xyz="0 0 0" rpy="0 0 0" />
@@ -47,13 +46,12 @@
       <visual>
         <geometry>
-          <mesh filename="package://mycobot_description/meshes/visual/joint2.dae" />
-        </geometry>
-        <origin xyz="0 0 0" rpy="0 0 0" />
-        <material name="white" />
-      </visual>
-      <collision>
-        <geometry>
-          <mesh filename="package://mycobot_description/meshes/visual/joint2.dae" />
-          <!-- <mesh filename="package://mycobot_description/meshes/collision/link2.stl" /> -->
+          <mesh filename="package://mycobot_description/meshes/visual/link2.dae" />
+        </geometry>
+        <origin xyz="0 0 0" rpy="0 0 0" />
+        <material name="white" />
+      </visual>
+      <collision>
+        <geometry>
+          <mesh filename="package://mycobot_description/meshes/collision/link2.stl" />
         </geometry>
         <origin xyz="0 0 0" rpy="0 0 0" />
@@ -68,13 +66,12 @@
       <visual>
         <geometry>
-          <mesh filename="package://mycobot_description/meshes/visual/joint3.dae" />
-        </geometry>
-        <origin xyz="0 0 0" rpy="0 0 0" />
-        <material name="white" />
-      </visual>
-      <collision>
-        <geometry>
-          <mesh filename="package://mycobot_description/meshes/visual/joint3.dae" />
-          <!-- <mesh filename="package://mycobot_description/meshes/collision/link3.stl" /> -->
+          <mesh filename="package://mycobot_description/meshes/visual/link3.dae" />
+        </geometry>
+        <origin xyz="0 0 0" rpy="0 0 0" />
+        <material name="white" />
+      </visual>
+      <collision>
+        <geometry>
+          <mesh filename="package://mycobot_description/meshes/collision/link3.stl" />
         </geometry>
         <origin xyz="0 0 0" rpy="0 0 0" />
@@ -89,13 +86,12 @@
       <visual>
         <geometry>
-          <mesh filename="package://mycobot_description/meshes/visual/joint4.dae" />
-        </geometry>
-        <origin xyz="0 0 0" rpy="0 0 0" />
-        <material name="white" />
-      </visual>
-      <collision>
-        <geometry>
-          <mesh filename="package://mycobot_description/meshes/visual/joint4.dae" />
-          <!-- <mesh filename="package://mycobot_description/meshes/collision/link4.stl" /> -->
+          <mesh filename="package://mycobot_description/meshes/visual/link4.dae" />
+        </geometry>
+        <origin xyz="0 0 0" rpy="0 0 0" />
+        <material name="white" />
+      </visual>
+      <collision>
+        <geometry>
+          <mesh filename="package://mycobot_description/meshes/collision/link4.stl" />
         </geometry>
         <origin xyz="0 0 0" rpy="0 0 0" />
@@ -110,13 +106,12 @@
       <visual>
         <geometry>
-          <mesh filename="package://mycobot_description/meshes/visual/joint5.dae" />
-        </geometry>
-        <origin xyz="0 0 0" rpy="0 0 0" />
-        <material name="white" />
-      </visual>
-      <collision>
-        <geometry>
-          <mesh filename="package://mycobot_description/meshes/visual/joint5.dae" />
-          <!-- <mesh filename="package://mycobot_description/meshes/collision/link5.stl" /> -->
+          <mesh filename="package://mycobot_description/meshes/visual/link5.dae" />
+        </geometry>
+        <origin xyz="0 0 0" rpy="0 0 0" />
+        <material name="white" />
+      </visual>
+      <collision>
+        <geometry>
+          <mesh filename="package://mycobot_description/meshes/collision/link5.stl" />
         </geometry>
         <origin xyz="0 0 0" rpy="0 0 0" />
@@ -131,5 +126,5 @@
       <visual>
         <geometry>
-          <mesh filename="package://mycobot_description/meshes/visual/joint6.dae" />
+          <mesh filename="package://mycobot_description/meshes/visual/link6.dae" />
         </geometry>
         <origin xyz="0 0 0 " rpy="0 0 0" />
@@ -138,6 +133,5 @@
       <collision>
         <geometry>
-          <mesh filename="package://mycobot_description/meshes/visual/joint6.dae" />
-          <!-- <mesh filename="package://mycobot_description/meshes/collision/link6.stl" /> -->
+          <mesh filename="package://mycobot_description/meshes/collision/link6.stl" />
         </geometry>
         <origin xyz="0 0 0" rpy="0 0 0" />
@@ -152,14 +146,11 @@
       <visual>
         <geometry>
-          <mesh filename="package://mycobot_description/meshes/visual/joint7.dae" />
-          <!-- <cylinder length="0.005" radius="0.02" /> -->
-        </geometry>
-        <origin xyz="0 0 0" rpy="0 0 0" />
-        <!-- <origin xyz="0 0 0" rpy="0 0 0" /> -->
-        <material name="white" />
-      </visual>
-      <collision>
-        <geometry>
-          <!-- <mesh filename="package://mycobot_description/meshes/collision/link6.stl" /> -->
+          <mesh filename="package://mycobot_description/meshes/visual/link7.dae" />
+        </geometry>
+        <origin xyz="0 0 0" rpy="0 0 0" />
+        <material name="white" />
+      </visual>
+      <collision>
+        <geometry>
           <cylinder length="0.0137" radius="0.0192" />
         </geometry>
@@ -193,5 +184,4 @@
       <parent link="${mycobot_link_3}" />
       <child link="${mycobot_link_4}" />
-      <!-- <origin xyz=" 0.00272 0 0.1104" rpy="0 0 0" /> -->
       <origin xyz=" 0 0 0.1104" rpy="0 0 0" />
       <dynamics damping="1.0e-6" friction="2.0e-1" />
@@ -202,6 +192,4 @@
       <parent link="${mycobot_link_4}" />
       <child link="${mycobot_link_5}" />
-      <!-- <origin xyz="-0.00164 0 0.096" rpy="0 0 0" /> -->
-      <!-- <origin xyz="0 0 0.096" rpy="0 0 0" /> -->
       <origin xyz="0 0 0.0965" rpy="0 0 0" />
       <dynamics damping="1.0e-6" friction="2.0e-1" />
@@ -212,5 +200,4 @@
       <parent link="${mycobot_link_5}" />
       <child link="${mycobot_link_6}" />
-      <!-- <origin xyz="0 0.0298 0.02876" rpy="0 0 0" /> -->
       <origin xyz="0 0.0335 0.034" rpy="0 0 0" />
       <dynamics damping="1.0e-6" friction="2.0e-1" />
@@ -221,5 +208,4 @@
       <parent link="${mycobot_link_6}" />
       <child link="${mycobot_link_7}" />
-      <!-- <origin xyz="-0.0456 0 0.03792" rpy="0 0 0" /> -->
       <origin xyz="-0.035 0 0.03792" rpy="0 0 0" />
       <dynamics damping="1.0e-6" friction="2.0e-1" />

Commit message: fixed the inertia of link4

File: mycobot_description/urdf/mycobot.xacro (robot description, xacro)
@@ -93,5 +93,5 @@
       </collision>
       <inertial>
-        <origin xyz="0 0.03 0.05" rpy="0 0 0" />
+        <origin xyz="0 -0.03 0.05" rpy="0 0 0" />
         <mass value="0.35" />
         <xacro:cylinder_inertia m="0.35" r="0.022" h="0.137" />
