Commit message: fixed inertia

File: mycobot_description/urdf/mycobot.urdf.xacro (robot description, xacro)
@@ -30,7 +30,7 @@
     </collision>
     <inertial>
-      <origin xyz="0 0 0" rpy="0 0 0" />
-      <mass value="1.0" />
-      <xacro:cylinder_inertia m="0.01" r="0.05" h="0.001" />
+      <origin xyz="0 0 0.003" rpy="0 0 0" />
+      <mass value="0.01" />
+      <xacro:cylinder_inertia m="0.01" r="0.05" h="0.006" />
     </inertial>
   </link>

File: mycobot_description/urdf/mycobot.xacro (robot description, xacro)
@@ -31,8 +31,8 @@
         <material name="white" />
       </visual>
-      <!-- <collision>
+      <collision>
         <geometry>
           <mesh filename="package://mycobot_description/meshes/visual/joint1.dae" />
-          <mesh filename="package://mycobot_description/meshes/collision/link1.stl" />
+          <!-- <mesh filename="package://mycobot_description/meshes/collision/link1.stl" /> -->
         </geometry>
         <origin xyz="0 0 0" rpy="0 0 0" />
@@ -42,5 +42,5 @@
         <mass value="1.0" />
         <xacro:cylinder_inertia m="1.0" r="0.05" h="0.07" />
-      </inertial> -->
+      </inertial>
     </link>
     <link name="${mycobot_link_2}">
@@ -52,16 +52,16 @@
         <material name="white" />
       </visual>
-      <!-- <collision>
+      <collision>
         <geometry>
           <mesh filename="package://mycobot_description/meshes/visual/joint2.dae" />
-          <mesh filename="package://mycobot_description/meshes/collision/link2.stl" />
-        </geometry>
-        <origin xyz="0 0 0" rpy="0 0 0" />
-      </collision>
-      <inertial>
-        <origin xyz="0 0 0.060" rpy="0 0 0" />
+          <!-- <mesh filename="package://mycobot_description/meshes/collision/link2.stl" /> -->
+        </geometry>
+        <origin xyz="0 0 0" rpy="0 0 0" />
+      </collision>
+      <inertial>
+        <origin xyz="0 0 0.04" rpy="0 0 0" />
         <mass value="0.2" />
-        <xacro:cylinder_inertia m="0.2" r="0.05" h="0.08" />
-      </inertial> -->
+        <xacro:cylinder_inertia m="0.2" r="0.025" h="0.08" />
+      </inertial>
     </link>
     <link name="${mycobot_link_3}">
@@ -73,16 +73,16 @@
         <material name="white" />
       </visual>
-      <!-- <collision>
+      <collision>
         <geometry>
           <mesh filename="package://mycobot_description/meshes/visual/joint3.dae" />
-          <mesh filename="package://mycobot_description/meshes/collision/link3.stl" />
-        </geometry>
-        <origin xyz="0 0 0" rpy="0 0 0" />
-      </collision>
-      <inertial>
-        <origin xyz="0.01 0 0.06" rpy="0 0 0" />
+          <!-- <mesh filename="package://mycobot_description/meshes/collision/link3.stl" /> -->
+        </geometry>
+        <origin xyz="0 0 0" rpy="0 0 0" />
+      </collision>
+      <inertial>
+        <origin xyz="0 0.03 0.06" rpy="0 0 0" />
         <mass value="0.4" />
-        <xacro:cylinder_inertia m="0.4" r="0.05" h="0.155" />
-      </inertial> -->
+        <xacro:cylinder_inertia m="0.4" r="0.025" h="0.155" />
+      </inertial>
     </link>
     <link name="${mycobot_link_4}">
@@ -94,16 +94,16 @@
         <material name="white" />
       </visual>
-      <!-- <collision>
+      <collision>
         <geometry>
           <mesh filename="package://mycobot_description/meshes/visual/joint4.dae" />
-          <mesh filename="package://mycobot_description/meshes/collision/link4.stl" />
-        </geometry>
-        <origin xyz="0 0 0" rpy="0 0 0" />
-      </collision>
-      <inertial>
-        <origin xyz="-0.01 0 0.05" rpy="0 0 0" />
-        <mass value="0.4" />
-        <xacro:cylinder_inertia m="0.4" r="0.05" h="0.155" />
-      </inertial> -->
+          <!-- <mesh filename="package://mycobot_description/meshes/collision/link4.stl" /> -->
+        </geometry>
+        <origin xyz="0 0 0" rpy="0 0 0" />
+      </collision>
+      <inertial>
+        <origin xyz="0 0.03 0.05" rpy="0 0 0" />
+        <mass value="0.35" />
+        <xacro:cylinder_inertia m="0.35" r="0.022" h="0.137" />
+      </inertial>
     </link>
     <link name="${mycobot_link_5}">
@@ -115,16 +115,16 @@
         <material name="white" />
       </visual>
-      <!-- <collision>
+      <collision>
         <geometry>
           <mesh filename="package://mycobot_description/meshes/visual/joint5.dae" />
-          <mesh filename="package://mycobot_description/meshes/collision/link5.stl" />
-        </geometry>
-        <origin xyz="0 0 0" rpy="0 0 0" />
-      </collision>
-      <inertial>
-        <origin xyz="0 0 0.05" rpy="0 0 0" />
+          <!-- <mesh filename="package://mycobot_description/meshes/collision/link5.stl" /> -->
+        </geometry>
+        <origin xyz="0 0 0" rpy="0 0 0" />
+      </collision>
+      <inertial>
+        <origin xyz="0 0.03 0.01" rpy="0 0 0" />
         <mass value="0.2" />
-        <xacro:cylinder_inertia m="0.2" r="0.05" h="0.05" />
-      </inertial> -->
+        <xacro:cylinder_inertia m="0.2" r="0.025" h="0.05" />
+      </inertial>
     </link>
     <link name="${mycobot_link_6}">
@@ -136,8 +136,8 @@
         <material name="white" />
       </visual>
-      <!-- <collision>
+      <collision>
         <geometry>
           <mesh filename="package://mycobot_description/meshes/visual/joint6.dae" />
-          <mesh filename="package://mycobot_description/meshes/collision/link6.stl" />
+          <!-- <mesh filename="package://mycobot_description/meshes/collision/link6.stl" /> -->
         </geometry>
         <origin xyz="0 0 0" rpy="0 0 0" />
@@ -146,6 +146,6 @@
         <origin xyz="0 0 0.037" rpy="0 0 0" />
         <mass value="0.5" />
-        <xacro:cylinder_inertia m="0.5" r="0.05" h="0.06" />
-      </inertial> -->
+        <xacro:cylinder_inertia m="0.5" r="0.025" h="0.06" />
+      </inertial>
     </link>
     <link name="${mycobot_link_7}">
@@ -159,16 +159,16 @@
         <material name="white" />
       </visual>
-      <!-- <collision>
-        <geometry>
-          <mesh filename="package://mycobot_description/meshes/visual/joint7.dae" />
-          <cylinder length="0.005" radius="0.02" />
-        </geometry>
-        <origin xyz="0 0 0" rpy="0 0 0" />
-      </collision>
-      <inertial>
-        <origin xyz="0 0.0025 0" rpy="${M_PI/2} 0 0" />
+      <collision>
+        <geometry>
+          <!-- <mesh filename="package://mycobot_description/meshes/collision/link6.stl" /> -->
+          <cylinder length="0.0137" radius="0.0192" />
+        </geometry>
+        <origin xyz="-0.00685 0 0" rpy="0 -${M_PI/2} 0" />
+      </collision>
+      <inertial>
+        <origin xyz="-0.005 0 0" rpy="0 -${M_PI/2} 0" />
         <mass value="0.1" />
-        <xacro:cylinder_inertia m="0.1" r="0.02" h="0.005" />
-      </inertial> -->
+        <xacro:cylinder_inertia m="0.1" r="0.02" h="0.01" />
+      </inertial>
     </link>
     <joint name="${mycobot_joint_1}" type="revolute">
@@ -305,5 +305,5 @@
         </actuator>
       </transmission>
-      <gazebo reference="${mycobot_link_1}">
+      <!-- <gazebo reference="${mycobot_link_1}">
         <material>Gazebo/White</material>
       </gazebo>
@@ -322,5 +322,5 @@
       <gazebo reference="${mycobot_link_6}">
         <material>Gazebo/White</material>
-      </gazebo>
+      </gazebo> -->
     </xacro:if>
   </xacro:macro>

Commit message: changed package name

File: mycobot_description/urdf/mycobot.urdf.xacro (robot description, xacro)
@@ -25,5 +25,5 @@
     <collision>
       <geometry>
-        <mesh filename="package://mycobot_description/meshes/visual/base_link.dae" />
+        <mesh filename="package://mycobot_description/meshes/collision/base_link.stl" />
       </geometry>
       <origin xyz="0 0 0" rpy="0 0 0" />

Commit message: modified trivials

File: mycobot_description/urdf/mycobot.urdf.xacro (robot description, xacro)
@@ -21,5 +21,4 @@
       </geometry>
       <origin xyz="0 0 0" rpy="0 0 0" />
-      <material name="white" />
     </visual>
     <collision>

File: mycobot_description/urdf/mycobot.xacro (robot description, xacro)
@@ -2,5 +2,4 @@
 <robot xmlns:xacro="http://ros.org/wiki/xacro">
   <xacro:include filename="$(find mycobot_description)/urdf/common.xacro" />
-  <xacro:include filename="$(find mycobot_description)/urdf/color.xacro" />
   <xacro:macro name="mycobot_robot" params="prefix parent *joint_origin">
     <xacro:property name="mycobot_link_1" value="${prefix}link1" />
@@ -29,5 +28,4 @@
         </geometry>
         <origin xyz="0 0 0" rpy="0 0 0" />
-        <material name="white" />
       </visual>
       <collision>
@@ -49,5 +47,4 @@
         </geometry>
         <origin xyz="0 0 0" rpy="0 0 0" />
-        <material name="white" />
       </visual>
       <collision>
@@ -69,5 +66,4 @@
         </geometry>
         <origin xyz="0 0 0" rpy="0 0 0" />
-        <material name="white" />
       </visual>
       <collision>
@@ -89,5 +85,4 @@
         </geometry>
         <origin xyz="0 0 0" rpy="0 0 0" />
-        <material name="white" />
       </visual>
       <collision>
@@ -109,5 +104,4 @@
         </geometry>
         <origin xyz="0 0 0" rpy="0 0 0" />
-        <material name="white" />
       </visual>
       <collision>
@@ -129,5 +123,4 @@
         </geometry>
         <origin xyz="0 0 0 " rpy="0 0 0" />
-        <material name="white" />
       </visual>
       <collision>
@@ -149,5 +142,4 @@
         </geometry>
         <origin xyz="0 0 0" rpy="0 0 0" />
-        <material name="white" />
       </visual>
       <collision>
@@ -291,22 +283,4 @@
         </actuator>
       </transmission>
-      <!-- <gazebo reference="${mycobot_link_1}">
-        <material>Gazebo/White</material>
-      </gazebo>
-      <gazebo reference="${mycobot_link_2}">
-        <material>Gazebo/White</material>
-      </gazebo>
-      <gazebo reference="${mycobot_link_3}">
-        <material>Gazebo/White</material>
-      </gazebo>
-      <gazebo reference="${mycobot_link_4}">
-        <material>Gazebo/White</material>
-      </gazebo>
-      <gazebo reference="${mycobot_link_5}">
-        <material>Gazebo/White</material>
-      </gazebo>
-      <gazebo reference="${mycobot_link_6}">
-        <material>Gazebo/White</material>
-      </gazebo> -->
     </xacro:if>
   </xacro:macro>

Commit message: add gripper in urdf

File: mycobot_description/urdf/mycobot.urdf.xacro (robot description, xacro)
@@ -8,4 +8,9 @@
   <xacro:arg name="robot_namespace" default="" />
   <xacro:arg name="virtual_base_link" default="false" />
+  <xacro:arg name="hand" default="true" />
+  <xacro:if value="$(arg hand)">
+    <xacro:include filename="$(find mycobot_description)/urdf/hand.xacro"/>
+    <xacro:hand connected_to="link6_flange" xyz='-0.015 0 0'/>
+  </xacro:if>
   <xacro:include filename="$(find mycobot_description)/urdf/mycobot.xacro" />
   <!-- Used for fixing robot to Gazebo 'base_link' -->
@@ -35,5 +40,5 @@
   </link>
   <xacro:property name="mycobot_origin" value="0 0 0.006" />
-  <xacro:mycobot_robot prefix="" parent="base_link">
+  <xacro:mycobot_robot parent="base_link">
     <origin xyz="${mycobot_origin}" rpy="0 0 0" />
   </xacro:mycobot_robot>

File: mycobot_description/urdf/mycobot.xacro (robot description, xacro)
@@ -2,18 +2,18 @@
 <robot xmlns:xacro="http://ros.org/wiki/xacro">
   <xacro:include filename="$(find mycobot_description)/urdf/common.xacro" />
-  <xacro:macro name="mycobot_robot" params="prefix parent *joint_origin">
-    <xacro:property name="mycobot_link_1" value="${prefix}link1" />
-    <xacro:property name="mycobot_link_2" value="${prefix}link2" />
-    <xacro:property name="mycobot_link_3" value="${prefix}link3" />
-    <xacro:property name="mycobot_link_4" value="${prefix}link4" />
-    <xacro:property name="mycobot_link_5" value="${prefix}link5" />
-    <xacro:property name="mycobot_link_6" value="${prefix}link6" />
-    <xacro:property name="mycobot_link_7" value="${prefix}link6_flange" />
-    <xacro:property name="mycobot_joint_1" value="${prefix}joint1" />
-    <xacro:property name="mycobot_joint_2" value="${prefix}joint2" />
-    <xacro:property name="mycobot_joint_3" value="${prefix}joint3" />
-    <xacro:property name="mycobot_joint_4" value="${prefix}joint4" />
-    <xacro:property name="mycobot_joint_5" value="${prefix}joint5" />
-    <xacro:property name="mycobot_joint_6" value="${prefix}joint6" />
+  <xacro:macro name="mycobot_robot" params="parent *joint_origin">
+    <xacro:property name="mycobot_link_1" value="link1" />
+    <xacro:property name="mycobot_link_2" value="link2" />
+    <xacro:property name="mycobot_link_3" value="link3" />
+    <xacro:property name="mycobot_link_4" value="link4" />
+    <xacro:property name="mycobot_link_5" value="link5" />
+    <xacro:property name="mycobot_link_6" value="link6" />
+    <xacro:property name="mycobot_link_7" value="link6_flange" />
+    <xacro:property name="mycobot_joint_1" value="joint1" />
+    <xacro:property name="mycobot_joint_2" value="joint2" />
+    <xacro:property name="mycobot_joint_3" value="joint3" />
+    <xacro:property name="mycobot_joint_4" value="joint4" />
+    <xacro:property name="mycobot_joint_5" value="joint5" />
+    <xacro:property name="mycobot_joint_6" value="joint6" />
     <xacro:property name="joint_velocity_limit" value="1.0" />
     <joint name="base_joint" type="fixed">
