Commit message: applied gripper in gazebo

File: mycobot_description/urdf/hand.xacro (robot description, xacro)
@@ -3,5 +3,5 @@
   <xacro:macro name="hand" params="connected_to:='' rpy:='0 0 0' xyz:='0 0 0'">
     <xacro:unless value="${connected_to == ''}">
-      <joint name="$hand_joint" type="fixed">
+      <joint name="hand_joint" type="fixed">
         <parent link="${connected_to}"/>
         <child link="hand"/>
@@ -105,4 +105,5 @@
         <mu2>0.2</mu2>
         <selfCollide>true</selfCollide>
+        <material>Gazebo/Pedestrian</material>
       </gazebo>
       <gazebo reference="leftfinger">
@@ -110,4 +111,8 @@
         <mu2>0.2</mu2>
         <selfCollide>true</selfCollide>
+        <material>Gazebo/Pedestrian</material>
+      </gazebo>
+      <gazebo reference="hand">
+        <material>Gazebo/Residential</material>
       </gazebo>
     </xacro:if>
